Commit message: panda URDF decreased from 7 dof to 6

File: models/panda.urdf (robot description, URDF)
Before this commit: robot panda, 18 links, 17 joints
Joints:
- joint panda_joint7: type revolute -> fixed

Commit message: panda model unnecessary links deleted

File: models/panda.urdf (robot description, URDF)
Before this commit: robot panda, 18 links, 17 joints
Links:
- removed link panda_link0_sc
- removed link panda_link1_sc
- removed link panda_link2_sc
- removed link panda_link3_sc
- removed link panda_link4_sc
- removed link panda_link5_sc
- removed link panda_link6_sc
- removed link panda_link7_sc
Joints:
- removed joint panda_link0_sc_joint
- removed joint panda_link1_sc_joint
- removed joint panda_link2_sc_joint
- removed joint panda_link3_sc_joint
- removed joint panda_link4_sc_joint
- removed joint panda_link5_sc_joint
- removed joint panda_link6_sc_joint
- removed joint panda_link7_sc_joint
